File: interfaces.sch (KiCad schematic (older format))
At the start: 0 parts

Commit message: update,
Parts:
- added U?: FC-40P-LCD, symbol taobao-components:FC-40P-LCD
Connections:
- net labels added: +3V3, GND, LCD_CLK, LCD_D10, LCD_D11, LCD_D12, LCD_D13, LCD_D14, LCD_D15, LCD_D18, LCD_D19, LCD_D2, LCD_D20, LCD_D21, LCD_D22, LCD_D23, LCD_D3, LCD_D4, LCD_D5, LCD_D6, LCD_D7, LCD_DE, LCD_HSYNC, LCD_VSYNC, TPX1, TPX2, TPY1, TPY2, VLED+, VLED-
- wire segments 0 -> 52

Commit message: update,
Parts:
- added C?: C106, symbol taobao-c:C106
- added C?: C106-50v, symbol taobao-c:C106-50v
- added C?: C104-50v, symbol taobao-c:C104-50v
- added D?: SD_1N5819_S4, symbol taobao-sd:SD_1N5819_S4
- added L?: L_2.2uH, symbol taobao-l:L_2.2uH
- added R?: R104, symbol taobao-r:R104
- added R?: R5R1, symbol taobao-r:R5R1
- added U?: PT4101, symbol taobao-components:PT4101
Connections:
- net labels added: +5V
- wire segments 52 -> 86
Other:
- moved on the sheet: U?

Commit message: update,
Parts:
- added U?: GD5F1GQ4UQY1G, symbol taobao-components:GD5F1GQ4UQY1G
- added U?: MX25L12835F, symbol taobao-components:MX25L12835F
Connections:
- net labels added: SPI_CS, SPI_MISO, SPI_MOSI, SPI_SCK
- wire segments 86 -> 108
Changed lines of the file:
@@
 Wire Wire Line
 	2000 8850 2050 8850
+$Comp
+L taobao-components:GD5F1GQ4UQY1G U?
+U 1 1 5BF2E5B6
+P 6800 9400
+F 0 "U?" H 6800 9850 50  0000 C CNN
+F 1 "GD5F1GQ4UQY1G" H 6800 9750 50  0000 C CNN
+F 2 "" H 6700 9350 50  0001 C CNN
+F 3 "" H 6700 9350 50  0001 C CNN
+	1    6800 9400
+	1    0    0    -1
+$EndComp
+$Comp
+L taobao-components:MX25L12835F U?
+U 1 1 5BF2E67C
+P 6800 8200
+F 0 "U?" H 6800 8700 50  0000 C CNN
+F 1 "MX25L12835F" H 6800 8600 50  0000 C CNN
+F 2 "" H 6700 8200 50  0001 C CNN
+F 3 "" H 6700 8200 50  0001 C CNN
+	1    6800 8200
+	1    0    0    -1
+$EndComp
+$Comp
+L customized_power:+3V3 #PWR?
+U 1 1 5BF2E710
+P 7500 7900
+F 0 "#PWR?" H 7500 7750 50  0001 C CNN
+F 1 "+3V3" H 7550 8100 50  0000 C CNN
+F 2 "" H 7500 7900 50  0001 C CNN
+F 3 "" H 7500 7900 50  0001 C CNN
+	1    7500 7900
+	1    0    0    -1
+$EndComp
+$Comp
+L customized_power:+3V3 #PWR?
+U 1 1 5BF2E738
+P 7500 9100
+F 0 "#PWR?" H 7500 8950 50  0001 C CNN
+F 1 "+3V3" H 7550 9300 50  0000 C CNN
+F 2 "" H 7500 9100 50  0001 C CNN
+F 3 "" H 7500 9100 50  0001 C CNN
+	1    7500 9100
+	1    0    0    -1
+$EndComp
+Wire Wire Line
+	7250 8050 7500 8050
+Wire Wire Line
+	7500 8050 7500 7900
+Wire Wire Line
+	7250 9250 7500 9250
+Wire Wire Line
+	7500 9250 7500 9100
+Wire Wire Line
+	7250 9350 7500 9350
+Wire Wire Line
+	7500 9350 7500 9250
+Connection ~ 7500 9250
+Wire Wire Line
+	7250 8150 7500 8150
+Wire Wire Line
+	7500 8150 7500 8050
+Connection ~ 7500 8050
+Text Label 7650 8250 2    50   ~ 0
+SPI_SCK
+Wire Wire Line
+	7650 8250 7250 8250
+Text Label 7650 8350 2    50   ~ 0
+SPI_MOSI
+Wire Wire Line
+	7650 8350 7250 8350
+Text Label 7650 9450 2    50   ~ 0
+SPI_SCK
+Wire Wire Line
+	7650 9450 7250 9450
+Text Label 7650 9550 2    50   ~ 0
+SPI_MOSI
+Wire Wire Line
+	7650 9550 7250 9550
+Text Label 5900 8050 0    50   ~ 0
+SPI_CS
+Wire Wire Line
+	5900 8050 6350 8050
+Text Label 5900 8150 0    50   ~ 0
+SPI_MISO
+Wire Wire Line
+	5900 8150 6350 8150
+$Comp
+L customized_power:+3V3 #PWR?
+U 1 1 5BF44176
+P 5900 8250
+F 0 "#PWR?" H 5900 8100 50  0001 C CNN
+F 1 "+3V3" V 5950 8400 50  0000 L CNN
+F 2 "" H 5900 8250 50  0001 C CNN
+F 3 "" H 5900 8250 50  0001 C CNN
+	1    5900 8250
+	0    -1   -1   0
+$EndComp
+Wire Wire Line
+	5900 8250 6350 8250
+$Comp
+L power:GND #PWR?
+U 1 1 5BF46D47
+P 6200 8450
+F 0 "#PWR?" H 6200 8200 50  0001 C CNN
+F 1 "GND" H 6250 8250 50  0000 C CNN
+F 2 "" H 6200 8450 50  0001 C CNN
+F 3 "" H 6200 8450 50  0001 C CNN
+	1    6200 8450
+	1    0    0    -1
+$EndComp
+Wire Wire Line
+	6200 8450 6200 8350
+Wire Wire Line
+	6200 8350 6350 8350
+Text Label 5900 9250 0    50   ~ 0
+SPI_CS
+Wire Wire Line
+	5900 9250 6350 9250
+Text Label 5900 9350 0    50   ~ 0
+SPI_MISO
+Wire Wire Line
+	5900 9350 6350 9350
+$Comp
+L customized_power:+3V3 #PWR?
+U 1 1 5BF49A01
+P 5900 9450
+F 0 "#PWR?" H 5900 9300 50  0001 C CNN
+F 1 "+3V3" V 5950 9600 50  0000 L CNN
+F 2 "" H 5900 9450 50  0001 C CNN
+F 3 "" H 5900 9450 50  0001 C CNN
+	1    5900 9450
+	0    -1   -1   0
+$EndComp
+Wire Wire Line
+	5900 9450 6350 9450
+$Comp
+L power:GND #PWR?
+U 1 1 5BF49A08
+P 6200 9650
+F 0 "#PWR?" H 6200 9400 50  0001 C CNN
+F 1 "GND" H 6250 9450 50  0000 C CNN
+F 2 "" H 6200 9650 50  0001 C CNN
+F 3 "" H 6200 9650 50  0001 C CNN
+	1    6200 9650
+	1    0    0    -1
+$EndComp
+Wire Wire Line
+	6200 9650 6200 9550
+Wire Wire Line
+	6200 9550 6350 9550
 $EndSCHEMATC

Commit message: update,
Parts:
- added C? (x2): C104, symbol taobao-c:C104
- added C?: C106, symbol taobao-c:C106
- added R? (x6): R473, symbol taobao-r:R473
- added U?: TF_CARD, symbol taobao-components:TF_CARD
- added U?: USB_MICRO, symbol taobao-components:USB_MICRO
Connections:
- net labels added: SDC0_CLK, SDC0_CMD, SDC0_D0, SDC0_D1, SDC0_D2, SDC0_D3, SDC0_Dn, USB_N, USB_P, VBUS
- wire segments 108 -> 166

Commit message: update,
Parts:
- added C?: C104, symbol taobao-c:C104
- added U?: NS2009, symbol taobao-components:NS2009
Connections:
- net labels added: PWNIRQ, TWI0_SCK, TWI0_SDA
- wire segments 166 -> 182
Other:
- moved on the sheet: C?, R?, U?

Commit message: update,
Connections:
- net labels added: LCD_Dn
Changed lines of the file:
@@
 Wire Wire Line
 	10500 3550 10500 3450
-Wire Bus Line
-	5750 5600 5750 6250
 Connection ~ 10500 3450
 Wire Wire Line
 	10500 3450 10850 3450
+Entry Wire Line
+	1550 5500 1650 5600
+Entry Wire Line
+	1550 5400 1650 5500
+Entry Wire Line
+	1550 5300 1650 5400
+Entry Wire Line
+	1550 5200 1650 5300
+Entry Wire Line
+	1550 5100 1650 5200
+Entry Wire Line
+	1550 5000 1650 5100
+Entry Wire Line
+	1550 4700 1650 4800
+Entry Wire Line
+	1550 4600 1650 4700
+Entry Wire Line
+	1550 4500 1650 4600
+Entry Wire Line
+	1550 4400 1650 4500
+Entry Wire Line
+	1550 4300 1650 4400
+Entry Wire Line
+	1550 4200 1650 4300
+Entry Wire Line
+	1550 3900 1650 4000
+Entry Wire Line
+	1550 3800 1650 3900
+Entry Wire Line
+	1550 3700 1650 3800
+Entry Wire Line
+	1550 3600 1650 3700
+Entry Wire Line
+	1550 3500 1650 3600
+Entry Wire Line
+	1550 3400 1650 3500
+Wire Bus Line
+	1550 2750 950  2750
+Wire Bus Line
+	5750 5600 5750 6250
+Wire Bus Line
+	1550 2750 1550 5500
+Text Label 1100 2750 0    50   ~ 0
+LCD_Dn
 $EndSCHEMATC

Commit message: update,
Parts:
- added R?: R103, symbol taobao-r:R103
Connections:
- wire segments 182 -> 184
Changed lines of the file:
@@
 Wire Bus Line
 	1550 2750 950  2750
+Text Label 1100 2750 0    50   ~ 0
+LCD_Dn
+$Comp
+L customized_power:+3V3 #PWR?
+U 1 1 5C3E281F
+P 8350 8600
+F 0 "#PWR?" H 8350 8450 50  0001 C CNN
+F 1 "+3V3" H 8400 8800 50  0000 C CNN
+F 2 "" H 8350 8600 50  0001 C CNN
+F 3 "" H 8350 8600 50  0001 C CNN
+	1    8350 8600
+	1    0    0    -1
+$EndComp
+$Comp
+L taobao-r:R103 R?
+U 1 1 5C3E2B0C
+P 8350 8900
+F 0 "R?" H 8450 8950 50  0000 L CNN
+F 1 "R103" H 8450 8900 50  0000 L CNN
+F 2 "" H 8350 8900 50  0001 C CNN
+F 3 "~" H 8350 8900 50  0001 C CNN
+	1    8350 8900
+	1    0    0    -1
+$EndComp
+Text Label 8350 9350 1    50   ~ 0
+SPI_CS
+Wire Wire Line
+	8350 8600 8350 8800
+Wire Wire Line
+	8350 9000 8350 9350
 Wire Bus Line
 	5750 5600 5750 6250
 Wire Bus Line
 	1550 2750 1550 5500
-Text Label 1100 2750 0    50   ~ 0
-LCD_Dn
 $EndSCHEMATC
