File: allwinner-v3s-tryout.sch (KiCad schematic (older format))
At the start: 0 parts

Commit message: update,
Changed lines of the file:
@@
 F0 "CPU" 50
 F1 "CPU.sch" 50
+F2 "LCD_Dn" I L 12500 7600 50
 $EndSheet
 $Sheet
@@
 F0 "interfaces" 50
 F1 "interfaces.sch" 50
+F2 "LCD_Dn" I R 11350 7600 50
 $EndSheet
+Wire Bus Line
+	11350 7600 12500 7600
 $EndSCHEMATC

Commit message: update,
Changed lines of the file:
@@
 EESchema Schematic File Version 4
-LIBS:I2C-adc-cache
+LIBS:allwinner-v3s-tryout-cache
 EELAYER 26 0
 EELAYER END
@@
 F0 "CPU" 50
 F1 "CPU.sch" 50
-F2 "LCD_Dn" I L 12500 7600 50
 $EndSheet
 $Sheet
@@
 F0 "interfaces" 50
 F1 "interfaces.sch" 50
-F2 "LCD_Dn" I R 11350 7600 50
 $EndSheet
-Wire Bus Line
-	11350 7600 12500 7600
 $EndSCHEMATC

Commit message: update,
Changed lines of the file:
@@
 $Descr A2 23386 16535
 encoding utf-8
-Sheet 1 5
+Sheet 1 2
 Title ""
 Date ""
@@
 F1 "CPU.sch" 50
 $EndSheet
-$Sheet
-S 12500 4850 1550 700
-U 5BCCA5FC
-F0 "power" 50
-F1 "power.sch" 50
-$EndSheet
-$Sheet
-S 9750 4850 1550 700
-U 5BCCA5FF
-F0 "media" 50
-F1 "media.sch" 50
-$EndSheet
-$Sheet
-S 9750 6150 1600 2400
-U 5BCCA602
-F0 "interfaces" 50
-F1 "interfaces.sch" 50
-$EndSheet
 $EndSCHEMATC
