File: power.sch (KiCad schematic (older format))
At the start: 0 parts

Commit message: update,
Parts:
- added R?: R0, symbol taobao-r:R0
Connections:
- new net +3V3: R?.2
- new net Vrtc: R?.1

Commit message: update,
Parts:
- added C? (x6): C106, symbol taobao-c:C106
- added C? (x3): C18pf, symbol taobao-c:C18pf
- added L? (x3): L_2.2uH, symbol taobao-l:L_2.2uH
- added R? (x3): R684, symbol taobao-r:R684
- added R? (x3): R154, symbol taobao-r:R154
- added U?: EA3036, symbol taobao-components:EA3036
Connections:
- net +3V3: now also C?.1, C?.1, C?.1, C?.1, C?.1, C?.1, L?.1, L?.1, L?.1, R?.1, R?.1, R?.1
- new net: L?.2, U?.11 (SW1)
- new net: C?.2, R?.2, R?.2, U?.14 (GND3)
- new net: C?.2, R?.2, R?.2, U?.2 (FB3)
- new net: L?.2, U?.20 (SW3)
- new net: C?.2, R?.2, R?.2, U?.3 (FB2)
- new net: L?.2, U?.6 (SW2)
- new net +5V: C?.2, C?.2, C?.2, U?.10 (VIN1), U?.16 (VIN3), U?.18 (EN3), U?.7 (VIN2), U?.8 (EN2), U?.9 (EN1)
- new net GND: C?.1, C?.1, C?.1, C?.2, C?.2, C?.2, R?.1, R?.1, R?.1, U?.12 (GND1), U?.13 (GND2), U?.14 (GND3), U?.15 (AGND), U?.17 (AGND), U?.21 (PAD), U?.4 (AGND)

Commit message: update,
Parts:
- added C?: C104, symbol taobao-c:C104
- added C?: C106, symbol taobao-c:C106
- added U?: XC6206, symbol taobao-components:XC6206
Connections:
- net +3V0: now also C?.1, C?.1, U?.2 (Vout)
- net +3V3: now also U?.3 (Vin)
- net GND: now also C?.2, C?.2, U?.1 (GND)
Changed lines of the file:
@@
 EELAYER 26 0
 EELAYER END
-$Descr A4 11693 8268
+$Descr A3 16535 11693
 encoding utf-8
 Sheet 3 5
@@
 Wire Wire Line
 	1500 4000 1500 4050
+$Comp
+L taobao-components:XC6206 U?
+U 1 1 5C0F1BEA
+P 3750 8300
+F 0 "U?" H 3750 8700 50  0000 C CNN
+F 1 "XC6206" H 3750 8600 50  0000 C CNN
+F 2 "" H 3750 7450 50  0001 C CNN
+F 3 "" H 3750 7450 50  0001 C CNN
+	1    3750 8300
+	1    0    0    -1
+$EndComp
+$Comp
+L customized_power:+3V3 #PWR?
+U 1 1 5C0F2036
+P 3050 8000
+F 0 "#PWR?" H 3050 7850 50  0001 C CNN
+F 1 "+3V3" H 3100 8200 50  0000 C CNN
+F 2 "" H 3050 8000 50  0001 C CNN
+F 3 "" H 3050 8000 50  0001 C CNN
+	1    3050 8000
+	1    0    0    -1
+$EndComp
+Wire Wire Line
+	3050 8000 3050 8150
+Wire Wire Line
+	3050 8150 3350 8150
+$Comp
+L power:GND #PWR?
+U 1 1 5C0F77BD
+P 3050 8900
+F 0 "#PWR?" H 3050 8650 50  0001 C CNN
+F 1 "GND" H 3100 8700 50  0000 C CNN
+F 2 "" H 3050 8900 50  0001 C CNN
+F 3 "" H 3050 8900 50  0001 C CNN
+	1    3050 8900
+	1    0    0    -1
+$EndComp
+Wire Wire Line
+	3050 8900 3050 8650
+Wire Wire Line
+	3050 8450 3350 8450
+$Comp
+L taobao-c:C104 C?
+U 1 1 5C0FD01C
+P 4300 8500
+F 0 "C?" H 4400 8550 50  0000 L CNN
+F 1 "C104" H 4400 8500 50  0000 L CNN
+F 2 "" H 4300 8500 50  0001 C CNN
+F 3 "~" H 4300 8500 50  0001 C CNN
+	1    4300 8500
+	1    0    0    -1
+$EndComp
+$Comp
+L taobao-c:C106 C?
+U 1 1 5C0FD0F4
+P 4700 8500
+F 0 "C?" H 4800 8550 50  0000 L CNN
+F 1 "C106" H 4800 8500 50  0000 L CNN
+F 2 "" H 4700 8500 50  0001 C CNN
+F 3 "~" H 4700 8500 50  0001 C CNN
+	1    4700 8500
+	1    0    0    -1
+$EndComp
+Wire Wire Line
+	4150 8300 4300 8300
+Wire Wire Line
+	4300 8300 4300 8400
+Wire Wire Line
+	4300 8300 4450 8300
+Wire Wire Line
+	4700 8300 4700 8400
+Connection ~ 4300 8300
+Wire Wire Line
+	4300 8600 4300 8650
+Connection ~ 3050 8650
+Wire Wire Line
+	3050 8650 3050 8450
+Wire Wire Line
+	4700 8600 4700 8650
+Wire Wire Line
+	3050 8650 4300 8650
+Connection ~ 4300 8650
+Wire Wire Line
+	4300 8650 4700 8650
+$Comp
+L taobao-components:+3V0 #PWR?
+U 1 1 5C11A42D
+P 4450 8200
+F 0 "#PWR?" H 4450 8050 50  0001 C CNN
+F 1 "+3V0" H 4500 8400 50  0000 C CNN
+F 2 "" H 4450 8200 50  0001 C CNN
+F 3 "" H 4450 8200 50  0001 C CNN
+	1    4450 8200
+	1    0    0    -1
+$EndComp
+Wire Wire Line
+	4450 8200 4450 8300
+Connection ~ 4450 8300
+Wire Wire Line
+	4450 8300 4700 8300
 $EndSCHEMATC

Commit message: update,
Parts:
- added C? (x8): C106, symbol taobao-c:C106
- added C? (x8): C105, symbol taobao-c:C105
- added C? (x6): C104, symbol taobao-c:C105
- added C? (x12): C104, symbol taobao-c:C104
- added R?: R204, symbol taobao-r:R204
- added R? (x2): R202, symbol taobao-r:R202
Connections:
- net +1V2: now also C?.1, C?.1, C?.1, C?.1, C?.1, C?.1, C?.1, C?.1, C?.1, C?.1, C?.1
- net +1V8: now also C?.1, C?.1, C?.1, C?.1, C?.1, C?.2, R?.2
- net +3V0: now also C?.1, C?.1, C?.1
- net +3V3: now also C?.1, C?.1, C?.1, C?.1, C?.1, C?.1, C?.1
- net GND: now also C?.1, C?.2, C?.2, C?.2, C?.2, C?.2, C?.2, C?.2, C?.2, C?.2, C?.2, C?.2, C?.2, C?.2, C?.2, C?.2, C?.2, C?.2, C?.2, C?.2, C?.2, C?.2, C?.2, C?.2, C?.2, C?.2, C?.2, C?.2, C?.2, C?.2, C?.2, C?.2, C?.2, R?.1, R?.2
- net Vrtc: now also C?.1
- new net: R?.1, R?.2
- new net SVREF: C?.1, C?.2
- new net VRA1: C?.1
- new net VRA2: C?.1, R?.1
- new net Vhp_bp: C?.1, C?.1
- new net Vrtc_io: C?.1

Commit message: update,
Changed lines of the file:
@@
 U 1 1 5C0A3AF9
 P 4650 3750
-F 0 "C?" V 4400 3750 50  0000 C CNN
-F 1 "C106" V 4500 3750 50  0000 C CNN
+F 0 "C?" V 4800 3750 50  0000 C CNN
+F 1 "C106" V 4900 3750 50  0000 C CNN
 F 2 "" H 4650 3750 50  0001 C CNN
 F 3 "~" H 4650 3750 50  0001 C CNN
@@
 U 1 1 5C0A4A70
 P 4650 4350
-F 0 "C?" V 4400 4350 50  0000 C CNN
-F 1 "C106" V 4500 4350 50  0000 C CNN
+F 0 "C?" V 4800 4350 50  0000 C CNN
+F 1 "C106" V 4900 4350 50  0000 C CNN
 F 2 "" H 4650 4350 50  0001 C CNN
 F 3 "~" H 4650 4350 50  0001 C CNN
@@
 U 1 1 5C0A5227
 P 4650 4950
-F 0 "C?" V 4400 4950 50  0000 C CNN
-F 1 "C106" V 4500 4950 50  0000 C CNN
+F 0 "C?" V 4450 4950 50  0000 C CNN
+F 1 "C106" V 4550 4950 50  0000 C CNN
 F 2 "" H 4650 4950 50  0001 C CNN
 F 3 "~" H 4650 4950 50  0001 C CNN
@@
 L customized_power:+5V #PWR?
 U 1 1 5C0A818B
-P 4600 5200
-F 0 "#PWR?" H 4600 5050 50  0001 C CNN
-F 1 "+5V" H 4700 5250 50  0000 L CNN
-F 2 "" H 4600 5200 50  0001 C CNN
-F 3 "" H 4600 5200 50  0001 C CNN
-	1    4600 5200
-	1    0    0    -1
+P 4850 5500
+F 0 "#PWR?" H 4850 5350 50  0001 C CNN
+F 1 "+5V" H 4950 5550 50  0000 L CNN
+F 2 "" H 4850 5500 50  0001 C CNN
+F 3 "" H 4850 5500 50  0001 C CNN
+	1    4850 5500
+	-1   0    0    1
 $EndComp
 Wire Wire Line
@@
 	4400 5200 4400 5250
 Wire Wire Line
-	4400 5250 4600 5250
+	4400 5250 4850 5250
 Wire Wire Line
-	4600 5250 4600 5200
+	4850 5250 4850 5500
 Connection ~ 4400 5250
 Wire Wire Line
