File: CPU.sch (KiCad schematic (older format))
At the start: 3 parts

Commit message: update,
Parts:
- added R?: R602, symbol taobao-r:R602
Connections:
- net labels added: AVCC, ETH_RX_N, ETH_RX_P, ETH_TX_N, ETH_TX_P, HBIAS, HP_COM, HP_COMFB, HP_L, HP_R, KEYADC0, LCD_Dn, MCSI_CK_N, MCSI_CK_P, MCSI_D0_N, MCSI_D0_P, MCSI_DI_N, MCSI_DI_P, MIC_N, MIC_P, PF6_USB_ID, SDC0_CLK, SDC0_CMD, SDC0_D0, SDC0_D1, SDC0_D2, SDC0_D3, SDC1_D3, USB_N, USB_P, VRA1, VRA2, VUSB, Vcc_phy, Vdd_phy, Vhp, Vhp_bp, Vmcsi, Vrtc, Vrtc_io, X32KIN, X32KOUT
- wire segments 120 -> 155

Commit message: update,
Connections:
- net labels added: SDC0_Dn
Changed lines of the file:
@@
 Text Label 7700 6450 0    50   ~ 0
 LCD_Dn
+Entry Wire Line
+	12550 3950 12650 3850
+Entry Wire Line
+	12650 3950 12750 3850
+Entry Wire Line
+	12950 3950 13050 3850
+Entry Wire Line
+	13050 3950 13150 3850
+Wire Bus Line
+	13200 3850 13200 3500
+Wire Bus Line
+	13200 3500 13650 3500
 Wire Bus Line
 	8100 5700 8100 6200
 Wire Bus Line
+	12650 3850 13200 3850
+Wire Bus Line
 	8100 6450 8100 9100
+Text Label 13300 3500 0    50   ~ 0
+SDC0_Dn
 $EndSCHEMATC

Commit message: update,
Parts:
- added C? (x4): C18pf, symbol taobao-c:C18pf
- added R?: R106, symbol taobao-r:R106
- added U?: MC-146, symbol taobao-components:MC-146
- added U?: XT_3225, symbol taobao-components:XT_3225
Connections:
- wire segments 155 -> 194
Other:
- moved on the sheet: R?, U?

Commit message: update,
Parts:
- added C?: C102, symbol taobao-c:C102
- added R?: R241, symbol taobao-r:R241
- added R?: R104, symbol taobao-r:R104
Connections:
- wire segments 194 -> 199
Other:
- moved on the sheet: C?, R?, U?

Commit message: update,
Connections:
- net labels removed: SDC0_Dn, SDC1_Dn
Changed lines of the file:
@@
 EESchema Schematic File Version 4
-LIBS:I2C-adc-cache
+LIBS:allwinner-v3s-tryout-cache
 EELAYER 26 0
 EELAYER END
@@
 Text Label 4050 4100 0    50   ~ 0
 SDC1_D0
-Entry Wire Line
-	3850 3800 3950 3900
-Entry Wire Line
-	3850 3900 3950 4000
-Entry Wire Line
-	3850 4000 3950 4100
-Wire Bus Line
-	3850 3500 3350 3500
-Text Label 3450 3500 0    50   ~ 0
-SDC1_Dn
 Text Label 4050 4200 0    50   ~ 0
 MCSI_PWDN
@@
 SDC0_D1
 Wire Wire Line
-	8500 1900 8500 2700
+	8500 2050 8500 2700
 $Comp
 L taobao-components:Vio #PWR?
 U 1 1 5BDFAC67
-P 8500 1900
-F 0 "#PWR?" H 8500 1750 50  0001 C CNN
-F 1 "Vio" V 8500 2050 50  0000 C CNN
-F 2 "" H 8500 1900 50  0001 C CNN
-F 3 "" H 8500 1900 50  0001 C CNN
-	1    8500 1900
-	1    0    0    -1
-$EndComp
-Wire Wire Line
-	8100 1900 8100 2700
+P 8500 2050
+F 0 "#PWR?" H 8500 1900 50  0001 C CNN
+F 1 "Vio" V 8500 2200 50  0000 C CNN
+F 2 "" H 8500 2050 50  0001 C CNN
+F 3 "" H 8500 2050 50  0001 C CNN
+	1    8500 2050
+	1    0    0    -1
+$EndComp
+Wire Wire Line
+	8100 2050 8100 2700
 $Comp
 L taobao-components:Vsys #PWR?
 U 1 1 5BE1A41F
-P 8100 1900
-F 0 "#PWR?" H 8100 1750 50  0001 C CNN
-F 1 "Vsys" V 8100 2100 50  0000 C CNN
-F 2 "" H 8100 1900 50  0001 C CNN
-F 3 "" H 8100 1900 50  0001 C CNN
-	1    8100 1900
-	1    0    0    -1
-$EndComp
-Wire Wire Line
-	8000 2100 8000 2700
+P 8100 2050
+F 0 "#PWR?" H 8100 1900 50  0001 C CNN
+F 1 "Vsys" V 8100 2250 50  0000 C CNN
+F 2 "" H 8100 2050 50  0001 C CNN
+F 3 "" H 8100 2050 50  0001 C CNN
+	1    8100 2050
+	1    0    0    -1
+$EndComp
+Wire Wire Line
+	8000 2400 8000 2700
 $Comp
 L customized_power:VUSB #PWR?
 U 1 1 5BE24F83
-P 8000 2100
-F 0 "#PWR?" H 8000 1950 50  0001 C CNN
-F 1 "VUSB" V 8000 2300 50  0000 C CNN
-F 2 "" H 8000 2100 50  0001 C CNN
-F 3 "" H 8000 2100 50  0001 C CNN
-	1    8000 2100
+P 8000 2400
+F 0 "#PWR?" H 8000 2250 50  0001 C CNN
+F 1 "VUSB" V 8000 2600 50  0000 C CNN
+F 2 "" H 8000 2400 50  0001 C CNN
+F 3 "" H 8000 2400 50  0001 C CNN
+	1    8000 2400
 	1    0    0    -1
 $EndComp
@@
 Wire Wire Line
 	6200 2150 6200 2700
-Wire Bus Line
-	6000 1650 5500 1650
-Text Label 5600 1650 0    50   ~ 0
-SDC1_Dn
-Entry Wire Line
-	6000 1650 6100 1750
-Entry Wire Line
-	3850 4300 3950 4400
-Entry Wire Line
-	3850 4400 3950 4500
-Entry Wire Line
-	3850 4800 3950 4900
-Entry Wire Line
-	3850 5000 3950 5100
-Entry Wire Line
-	3850 5100 3950 5200
-Entry Wire Line
-	3850 5200 3950 5300
-Entry Wire Line
-	3850 5300 3950 5400
-Entry Wire Line
-	3850 5400 3950 5500
-Entry Wire Line
-	3850 5500 3950 5600
-Entry Wire Line
-	3850 5900 3950 6000
-Entry Wire Line
-	3850 6000 3950 6100
-Entry Wire Line
-	3850 6100 3950 6200
-Entry Wire Line
-	3850 6400 3950 6500
-Entry Wire Line
-	3850 6500 3950 6600
-Entry Wire Line
-	3850 6700 3950 6800
-Entry Wire Line
-	3850 6800 3950 6900
-Entry Wire Line
-	3850 6900 3950 7000
-Wire Bus Line
-	3850 4250 3350 4250
-Text Label 3450 4250 0    50   ~ 0
-LCD_Dn
-Entry Wire Line
-	8300 1750 8400 1650
-Entry Wire Line
-	8400 1750 8500 1650
-Entry Wire Line
-	8700 1750 8800 1650
-Entry Wire Line
-	8800 1750 8900 1650
-Wire Bus Line
-	8950 1650 8950 1300
-Wire Bus Line
-	8950 1300 9400 1300
-Text Label 9050 1300 0    50   ~ 0
-SDC0_Dn
 $Comp
 L taobao-components:MC-146 U?
@@
 Text Label 1050 900  0    50   ~ 0
 LCD_Dn
-Wire Bus Line
-	3850 3500 3850 4000
-Wire Bus Line
-	8400 1650 8950 1650
-Wire Bus Line
-	3850 4250 3850 6900
+Text GLabel 3950 3900 0    50   Input ~ 0
+SDC1_D2
+Text GLabel 3950 4000 0    50   Input ~ 0
+SDC1_D1
+Text GLabel 3950 4100 0    50   Input ~ 0
+SDC1_D0
+Text GLabel 3950 4400 0    50   Input ~ 0
+LCD_D23
+Text GLabel 3950 4500 0    50   Input ~ 0
+LCD_D22
+Text GLabel 3950 4900 0    50   Input ~ 0
+LCD_D21
+Text GLabel 3950 5100 0    50   Input ~ 0
+LCD_D20
+Text GLabel 3950 5200 0    50   Input ~ 0
+LCD_D19
+Text GLabel 3950 5300 0    50   Input ~ 0
+LCD_D18
+Text GLabel 3950 5400 0    50   Input ~ 0
+LCD_D15
+Text GLabel 3950 5500 0    50   Input ~ 0
+LCD_D14
+Text GLabel 3950 5600 0    50   Input ~ 0
+LCD_D13
+Text GLabel 3950 6000 0    50   Input ~ 0
+LCD_D12
+Text GLabel 3950 6100 0    50   Input ~ 0
+LCD_D11
+Text GLabel 3950 6200 0    50   Input ~ 0
+LCD_D10
+Text GLabel 3950 6500 0    50   Input ~ 0
+LCD_D7
+Text GLabel 3950 6600 0    50   Input ~ 0
+LCD_D6
+Text GLabel 3950 6800 0    50   Input ~ 0
+LCD_D5
+Text GLabel 3950 6900 0    50   Input ~ 0
+LCD_D4
+Text GLabel 3950 7000 0    50   Input ~ 0
+LCD_D3
+Text GLabel 6100 1750 1    50   Input ~ 0
+SDC1_D3
+Text GLabel 8200 1750 1    50   Input ~ 0
+SDC0_D1
+Text GLabel 8300 1750 1    50   Input ~ 0
+SDC0_D0
+Text GLabel 8400 1750 1    50   Input ~ 0
+SDC0_CLK
+Text GLabel 8600 1750 1    50   Input ~ 0
+SDC0_CMD
+Text GLabel 8700 1750 1    50   Input ~ 0
+SDC0_D3
+Text GLabel 8800 1750 1    50   Input ~ 0
+SDC0_D2
 $EndSCHEMATC

Commit message: update,
Parts:
- added C? (x17): C106, symbol taobao-c:C106
- added C?: C106-50v, symbol taobao-c:C106-50v
- added C?: C104-50v, symbol taobao-c:C104-50v
- added C? (x16): C104, symbol taobao-c:C104
- added C? (x3): C18pf, symbol taobao-c:C18pf
- added C? (x8): C105, symbol taobao-c:C105
- added C? (x6): C104, symbol taobao-c:C105
- added D?: SD_1N5819_S4, symbol taobao-sd:SD_1N5819_S4
- added J? (x2): Conn_01x30, symbol Connector_Generic:Conn_01x30
- added L? (x4): L_2.2uH, symbol taobao-l:L_2.2uH
- added R?: R103, symbol taobao-r:R104
- added R?: R5R1, symbol taobao-r:R5R1
- added R? (x6): R473, symbol taobao-r:R473
- added R?: R103, symbol taobao-r:R103
- added R?: R0, symbol taobao-r:R0
- added R? (x3): R684, symbol taobao-r:R684
- added R? (x3): R154, symbol taobao-r:R154
- added R?: R204, symbol taobao-r:R204
- added R? (x2): R202, symbol taobao-r:R202
- added RN?: R_Pack04, symbol Device:R_Pack04
- added U?: FC-40P-LCD, symbol taobao-components:FC-40P-LCD
- added U?: PT4101, symbol taobao-components:PT4101
- added U?: GD5F1GQ4UQY1G, symbol taobao-components:GD5F1GQ4UQY1G
- added U?: MX25L12835F, symbol taobao-components:MX25L12835F
- added U?: TF_CARD, symbol taobao-components:TF_CARD
- added U?: USB_MICRO, symbol taobao-components:USB_MICRO
- added U?: NS2009, symbol taobao-components:NS2009
- added U?: EA3036, symbol taobao-components:EA3036
- added U?: XC6206, symbol taobao-components:XC6206
Connections:
- net labels added: +1V2, +1V8, +3V0, +5V, MCSI_D1_N, MCSI_D1_P, MCSI_DO_N, MCSI_DO_P, PENIRQ, PG0, PG1, PG2, PWM0, PWM1, SDC1_CLK, SDC1_CMD, TPX1, TPX2, TPY1, TPY2, TWI1_SCK0, TWI1_SDA0, UART1_RX, UART1_TX, UART2_CTS, UART2_RTS, USB_ID, VBUS, VLED+, VLED-, X32KOUT]
- wire segments 199 -> 746
Other:
- moved on the sheet: C?, R?

Commit message: update,
Connections:
- net MCSI_DI_N is gone; now on net MCSI_D1_N: U?.84 (MCSI-D1N)
- net MCSI_DI_P is gone; now on net MCSI_D1_P: U?.83 (MCSI-D1P)
- net TWI1_SCK: now also RN?.2 (R2.1)
- net TWI1_SCK0: no longer RN?.2 (R2.1)
- net TWI1_SDA: now also RN?.1 (R1.1)
- net TWI1_SDA0: no longer RN?.1 (R1.1)
- net MCSI_DO_N renamed MCSI_D0_N
- net MCSI_DO_P renamed MCSI_D0_P
Changed lines of the file:
@@
 MCSI_D0_N
 Text Label 11000 5100 2    50   ~ 0
-MCSI_DI_P
+MCSI_D1_P
 Text Label 11000 5000 2    50   ~ 0
-MCSI_DI_N
+MCSI_D1_N
 $Comp
 L taobao-components:Vmcsi #PWR?
@@
 MCSI_CK_P
 Text GLabel 11100 5000 2    50   Input ~ 0
-MCSI_DI_N
+MCSI_D1_N
 Text GLabel 11100 5100 2    50   Input ~ 0
-MCSI_DI_P
+MCSI_D1_P
 Text GLabel 11100 5200 2    50   Input ~ 0
-MCSI_DO_N
+MCSI_D0_N
 Text GLabel 11100 5300 2    50   Input ~ 0
-MCSI_DO_P
+MCSI_D0_P
 Text GLabel 11100 5600 2    50   Input ~ 0
 ETH_LED_SPD
@@
 Connection ~ 27400 13050
 Text Label 27400 14000 1    50   ~ 0
-TWI1_SDA0
+TWI1_SDA
 Wire Wire Line
 	27400 14000 27400 13500
 Text Label 27500 14000 1    50   ~ 0
-TWI1_SCK0
+TWI1_SCK
 Text Label 27600 14000 1    50   ~ 0
 TWI0_SDA
