File: CPU.sch (KiCad schematic (older format))
At the start: 102 parts

Commit message: update,
Connections:
- net PF6_USB_ID is gone; now on net USB_ID: R?.1, U?.100 (PF6), U?.4 (ID)
Changed lines of the file:
@@
 RESET
 Text Label 8900 2050 3    50   ~ 0
-PF6_USB_ID
+USB_ID
 Text Label 8800 2050 3    50   ~ 0
 SDC0_D2
@@
 USB_N
 Text GLabel 8900 1750 1    50   Input ~ 0
-PF6_USB_ID
+USB_ID
 Text GLabel 9000 1750 1    50   Input ~ 0
 RESET
@@
 USB_P
 Text GLabel 22600 2700 0    50   Input ~ 0
-PF6_USB_ID
+USB_ID
 $Comp
 L customized_power:+3V3 #PWR?
@@
 Wire Wire Line
 	27500 13500 27500 14000
+Text Label 8900 2550 1    50   ~ 0
+PF6
 $EndSCHEMATC
