File: CPU.sch (KiCad schematic (older format))
At the start: 102 parts

Commit message: update,
Parts:
- C1, C11, C12, C13, C14, C15, C16, C17, C18, C19, C2, C20, C21, C22, C23, C24, C25, C26, C27, C28, C29, C3, C30, C31, C32, C33, C34, C35, C36, C37, C38, C39, C4, C40, C41, C42, C43, C44, C45, C46, C47, C48, C49, C5, C50, C51, C52, C53, C54, C55, C56, C57, C58, C6, C7, C8: renamed from C?; footprint (none) -> Capacitor_SMD:C_0805_2012Metric_Pad1.15x1.40mm_HandSolder
- C10, C9: renamed from C?; footprint (none) -> Capacitor_SMD:C_1206_3216Metric_Pad1.42x1.75mm_HandSolder
- D1: renamed from D?; footprint (none) -> Diode_SMD:D_SOD-123F
- J1, J2: renamed from J?; footprint (none) -> footprint-lib.pretty:Pin_Header_Straight_1x30_Pitch2.54mm
- L1, L2, L3, L4: renamed from L?; footprint (none) -> Inductor_SMD:L_0805_2012Metric_Pad1.15x1.40mm_HandSolder
- R1, R10, R11, R12, R13, R14, R15, R16, R17, R18, R19, R2, R20, R21, R22, R23, R24, R3, R4, R5, R6, R7, R8, R9: renamed from R?; footprint (none) -> Resistor_SMD:R_0805_2012Metric_Pad1.15x1.40mm_HandSolder
- U1: renamed from U?; footprint (none) -> Connector_PinHeader_2.54mm:PinHeader_1x05_P2.54mm_Vertical
- U2: renamed from U?; footprint (none) -> Package_SO:MSOP-10_3x3mm_P0.5mm
- U4: renamed from U?; footprint (none) -> w_smd_lqfp:lqfp128
- gave numbers to parts that had none: 10

Commit message: update,
Changed lines of the file:
@@
 	1    0    0    -1
 $EndComp
-Text HLabel 1450 900  2    50   Input ~ 0
-LCD_Dn
-Wire Bus Line
-	1450 900  950  900
-Text Label 1050 900  0    50   ~ 0
-LCD_Dn
 Text GLabel 3950 3900 0    50   Input ~ 0
 SDC1_D2

Commit message: update,
Parts:
- removed RN1: R_Pack04, symbol Device:R_Pack04
- removed U10: GD5F1GQ4UQY1G, symbol taobao-components:GD5F1GQ4UQY1G
- added R25, R26, R27, R28: R202, Resistor_SMD:R_0603_1608Metric_Pad1.05x0.95mm_HandSolder, symbol taobao-r:R202
- added U10: GD5F1GQ4UAYIG, Package_SO:SOIC-8_3.9x4.9mm_P1.27mm, symbol taobao-components:GD5F1GQ4UAYIG
- U11: footprint (none) -> Package_DFN_QFN:QFN-24-1EP_3x3mm_P0.4mm_EP1.75x1.6mm_ThermalVias
- U12: footprint (none) -> Package_TO_SOT_SMD:SOT-23_Handsoldering
- U3: footprint (none) -> footprint-lib.pretty:HIROSE_FH12S-40S-0.5SH(55)
- U5: footprint (none) -> footprint-lib.pretty:SUNTECH_ST-TF-003A
- U6: footprint (none) -> Crystal:Crystal_SMD_SeikoEpson_MC146-4Pin_6.7x1.5mm_HandSoldering
- U7: footprint (none) -> Package_SO:SOIC-8_3.9x4.9mm_P1.27mm
- U8: footprint (none) -> Package_TO_SOT_SMD:SOT-23-6_Handsoldering
- U9: footprint (none) -> Crystal:Crystal_SMD_SeikoEpson_TSX3225-4Pin_3.2x2.5mm_HandSoldering
Connections:
- net +3V3: now also R25.1, R26.1, R27.1, R28.1, U10.3 (~WP~), U10.7 (~HOLD~), U10.8 (VCC)
- net GND: now also U10.4 (GND)
- net SPI_CS: now also U10.1 (~CS~)
- net SPI_MISO: now also U10.2 (SO)
- net SPI_MOSI: now also U10.5 (SI)
- net SPI_SCK: now also U10.6 (CLK)
- net TWI0_SCK: now also R28.2
- net TWI0_SDA: now also R27.2
- net TWI1_SCK: now also R26.2
- net TWI1_SDA: now also R25.2
Changed lines of the file:
@@
 F 0 "U6" H 13950 7600 50  0000 C CNN
 F 1 "MC-146" H 13950 7500 50  0000 C CNN
-F 2 "" H 14250 7200 50  0001 C CNN
+F 2 "Crystal:Crystal_SMD_SeikoEpson_MC146-4Pin_6.7x1.5mm_HandSoldering" H 14250 7200 50  0001 C CNN
 F 3 "" H 14250 7200 50  0001 C CNN
 	1    13950 7200
@@
 F 0 "U9" H 14450 8500 50  0000 C CNN
 F 1 "XT_3225" H 14450 8600 50  0000 C CNN
-F 2 "" H 14400 8950 50  0001 C CNN
+F 2 "Crystal:Crystal_SMD_SeikoEpson_TSX3225-4Pin_3.2x2.5mm_HandSoldering" H 14400 8950 50  0001 C CNN
 F 3 "" H 14400 8950 50  0001 C CNN
 	1    14450 8950
@@
 F 0 "U3" H 20100 4250 50  0000 L CNN
 F 1 "FC-40P-LCD" H 20100 4200 50  0000 L CNN
-F 2 "" H 18650 5250 50  0001 C CNN
+F 2 "footprint-lib.pretty:HIROSE_FH12S-40S-0.5SH(55)" H 18650 5250 50  0001 C CNN
 F 3 "" H 18650 5250 50  0001 C CNN
 	1    19900 4300
@@
 F 0 "U8" H 19250 8850 50  0000 C CNN
 F 1 "PT4101" H 19250 8750 50  0000 C CNN
-F 2 "" H 19250 8400 50  0001 C CNN
+F 2 "Package_TO_SOT_SMD:SOT-23-6_Handsoldering" H 19250 8400 50  0001 C CNN
 F 3 "" H 19250 8400 50  0001 C CNN
 	1    19250 8400
@@
 	18200 8250 18250 8250
 $Comp
-L taobao-components:GD5F1GQ4UQY1G U?
-U 1 1 5BFB141C
-P 24250 9750
-AR Path="/5BCCA602/5BFB141C" Ref="U?"  Part="1"
-AR Path="/5BCC9E7B/5BFB141C" Ref="U10"  Part="1"
-F 0 "U10" H 24250 10200 50  0000 C CNN
-F 1 "GD5F1GQ4UQY1G" H 24250 10100 50  0000 C CNN
-F 2 "" H 24150 9700 50  0001 C CNN
-F 3 "" H 24150 9700 50  0001 C CNN
-	1    24250 9750
-	1    0    0    -1
-$EndComp
-$Comp
 L taobao-components:MX25L12835F U?
 U 1 1 5BFB1423
@@
 F 0 "U7" H 24250 8350 50  0000 C CNN
 F 1 "MX25L12835F" H 24250 8250 50  0000 C CNN
-F 2 "" H 24150 7850 50  0001 C CNN
+F 2 "Package_SO:SOIC-8_3.9x4.9mm_P1.27mm" H 24150 7850 50  0001 C CNN
 F 3 "" H 24150 7850 50  0001 C CNN
 	1    24250 7850
@@
 F 0 "U5" H 23850 6450 50  0000 C CNN
 F 1 "TF_CARD" H 23850 6350 50  0000 C CNN
-F 2 "" H 23800 5650 50  0001 C CNN
+F 2 "footprint-lib.pretty:SUNTECH_ST-TF-003A" H 23800 5650 50  0001 C CNN
 F 3 "" H 23800 5650 50  0001 C CNN
 	1    23850 5650
@@
 F 0 "U11" H 4450 18450 50  0000 C CNN
 F 1 "EA3036" H 4450 18350 50  0000 C CNN
-F 2 "" H 4500 15100 50  0001 C CNN
+F 2 "Package_DFN_QFN:QFN-24-1EP_3x3mm_P0.4mm_EP1.75x1.6mm_ThermalVias" H 4500 15100 50  0001 C CNN
 F 3 "" H 4500 15100 50  0001 C CNN
 	1    4500 16300
@@
 F 0 "U12" H 4500 19650 50  0000 C CNN
 F 1 "XC6206" H 4500 19550 50  0000 C CNN
-F 2 "" H 4500 18400 50  0001 C CNN
+F 2 "Package_TO_SOT_SMD:SOT-23_Handsoldering" H 4500 18400 50  0001 C CNN
 F 3 "" H 4500 18400 50  0001 C CNN
 	1    4500 19250
@@
 	1    0    0    -1
 $EndComp
-$Comp
-L Device:R_Pack04 RN1
-U 1 1 5C8E5541
-P 27600 13300
-F 0 "RN1" H 27800 13350 50  0000 L CNN
-F 1 "R_Pack04" H 27800 13300 50  0000 L CNN
-F 2 "" V 27875 13300 50  0001 C CNN
-F 3 "~" H 27600 13300 50  0001 C CNN
-	1    27600 13300
-	1    0    0    -1
-$EndComp
 Wire Wire Line
 	27400 12850 27400 13050
 Wire Wire Line
 	27400 13050 27500 13050
-Wire Wire Line
-	27700 13050 27700 13100
-Wire Wire Line
-	27600 13100 27600 13050
 Connection ~ 27600 13050
 Wire Wire Line
 	27600 13050 27700 13050
-Wire Wire Line
-	27500 13100 27500 13050
 Connection ~ 27500 13050
 Wire Wire Line
 	27500 13050 27600 13050
-Wire Wire Line
-	27400 13100 27400 13050
 Connection ~ 27400 13050
 Text Label 27400 14000 1    50   ~ 0
 TWI1_SDA
-Wire Wire Line
-	27400 14000 27400 13500
 Text Label 27500 14000 1    50   ~ 0
 TWI1_SCK
@@
 Text Label 27700 14000 1    50   ~ 0
 TWI0_SCK
-Wire Wire Line
-	27700 14000 27700 13500
-Wire Wire Line
-	27600 13500 27600 14000
-Wire Wire Line
-	27500 13500 27500 14000
 Text Label 8900 2550 1    50   ~ 0
 PF6
 NoConn ~ 19100 5700
+$Comp
+L taobao-r:R202 R25
+U 1 1 5BDB1796
+P 27400 13300
+F 0 "R25" H 27500 13350 50  0000 L CNN
+F 1 "R202" H 27500 13300 50  0000 L CNN
+F 2 "Resistor_SMD:R_0603_1608Metric_Pad1.05x0.95mm_HandSolder" H 27400 13300 50  0001 C CNN
+F 3 "~" H 27400 13300 50  0001 C CNN
+	1    27400 13300
+	1    0    0    -1
+$EndComp
+$Comp
+L taobao-r:R202 R26
+U 1 1 5BDB1892
+P 27500 13300
+F 0 "R26" H 27600 13350 50  0000 L CNN
+F 1 "R202" H 27600 13300 50  0000 L CNN
+F 2 "Resistor_SMD:R_0603_1608Metric_Pad1.05x0.95mm_HandSolder" H 27500 13300 50  0001 C CNN
+F 3 "~" H 27500 13300 50  0001 C CNN
+	1    27500 13300
+	1    0    0    -1
+$EndComp
+$Comp
+L taobao-r:R202 R27
+U 1 1 5BDB1974
+P 27600 13300
+F 0 "R27" H 27700 13350 50  0000 L CNN
+F 1 "R202" H 27700 13300 50  0000 L CNN
+F 2 "Resistor_SMD:R_0603_1608Metric_Pad1.05x0.95mm_HandSolder" H 27600 13300 50  0001 C CNN
+F 3 "~" H 27600 13300 50  0001 C CNN
+	1    27600 13300
+	1    0    0    -1
+$EndComp
+$Comp
+L taobao-r:R202 R28
+U 1 1 5BDB1A54
+P 27700 13300
+F 0 "R28" H 27800 13350 50  0000 L CNN
+F 1 "R202" H 27800 13300 50  0000 L CNN
+F 2 "Resistor_SMD:R_0603_1608Metric_Pad1.05x0.95mm_HandSolder" H 27700 13300 50  0001 C CNN
+F 3 "~" H 27700 13300 50  0001 C CNN
+	1    27700 13300
+	1    0    0    -1
+$EndComp
+Wire Wire Line
+	27700 13050 27700 13200
+Wire Wire Line
+	27700 13400 27700 14000
+Wire Wire Line
+	27600 13050 27600 13200
+Wire Wire Line
+	27600 13400 27600 14000
+Wire Wire Line
+	27400 13050 27400 13200
+Wire Wire Line
+	27500 13050 27500 13200
+Wire Wire Line
+	27400 13400 27400 14000
+Wire Wire Line
+	27500 13400 27500 14000
+$Comp
+L taobao-components:GD5F1GQ4UAYIG U10
+U 1 1 5C50C62F
+P 24250 9750
+F 0 "U10" H 24250 10200 50  0000 C CNN
+F 1 "GD5F1GQ4UAYIG" H 24250 10100 50  0000 C CNN
+F 2 "Package_SO:SOIC-8_3.9x4.9mm_P1.27mm" H 24150 9700 50  0001 C CNN
+F 3 "" H 24150 9700 50  0001 C CNN
+	1    24250 9750
+	1    0    0    -1
+$EndComp
 $EndSCHEMATC

Commit message: update,
Parts:
- added C? (x4): C104, symbol taobao-c:C104
- added C?: C105, symbol taobao-c:C105
- added C? (x2): C33pf, symbol taobao-c:C33pf
- added C?: C101, symbol taobao-c:C101
- added L?: L_10uH, symbol taobao-l:L_10uH
- added MK?: Microphone, symbol Device:Microphone
- added R? (x4): R510, symbol taobao-r:R510
- added R? (x2): R202, symbol taobao-r:R202
- added R?: R682, symbol taobao-r:R682
- added R?: R822, symbol taobao-r:R822
- added R?: R103, symbol taobao-r:R103
- added R?: R113, symbol taobao-r:R113
- added SW? (x4): SW_Push, symbol Switch:SW_Push
- added U?: HR911105A, footprint-lib.pretty:HANRUN_HR911105A, symbol taobao-components:HR911105A
Connections:
- net +3V0: now also C?.1, R?.2
- net +3V3: now also L?.1
- net ETH_RX_N: now also R?.1, U?.6 (RD-)
- net ETH_RX_P: now also R?.1, U?.3 (RD+)
- net ETH_TX_N: now also R?.1, U?.2 (TD-)
- net ETH_TX_P: now also R?.1, U?.1 (TD+)
- net GND: now also C?.2, C?.2, C?.2, C?.2, C?.2, R?.2, SW?.2, SW?.2, SW?.2, SW?.2, U?.8 (CHS_GND)
- net KEYADC0: now also R?.2
- net MIC_N: now also C?.1
- net MIC_P: now also C?.1
- new net: C?.1, L?.2, R?.2, R?.2, U?.4 (TCT)
- new net: C?.1, R?.2, R?.2, U?.5 (TCT)
- new net: C?.1, C?.2, C?.2, MK?.1 (-), R?.1
- new net: C?.1, C?.1, C?.2, MK?.2 (+), R?.1
- new net: R?.1, R?.2, SW?.1 (x3)
- new net: R?.1, SW?.1

Commit message: update,
Parts:
- added J?: Conn_01x24, symbol Connector_Generic:Conn_01x24
- J1, J2: footprint footprint-lib.pretty:Pin_Header_Straight_1x30_Pitch2.54mm -> footprint-lib.pretty:Pin_Header_Straight_1x30_Pitch1.27mm
Connections:
- net +3V3: now also J?.2 (Pin_2)
- net +5V: now also J?.1 (Pin_1)
- net GND: now also J?.3 (Pin_3)
- net LCD_CLK: now also J?.21 (Pin_21)
- net LCD_D10: now also J?.8 (Pin_8)
- net LCD_D11: now also J?.9 (Pin_9)
- net LCD_D12: now also J?.6 (Pin_6)
- net LCD_D13: now also J?.7 (Pin_7)
- net LCD_D14: now also J?.4 (Pin_4)
- net LCD_D15: now also J?.5 (Pin_5)
- net LCD_D18: now also J?.22 (Pin_22)
- net LCD_D2: now also J?.14 (Pin_14)
- net LCD_D3: now also J?.15 (Pin_15)
- net LCD_D4: now also J?.12 (Pin_12)
- net LCD_D5: now also J?.13 (Pin_13)
- net LCD_D6: now also J?.10 (Pin_10)
- net LCD_D7: now also J?.11 (Pin_11)
- net LCD_DE: now also J?.20 (Pin_20)
- net LCD_HSYNC: now also J?.17 (Pin_17)
- net LCD_VSYNC: now also J?.16 (Pin_16)
- net TWI1_SCK: now also J?.19 (Pin_19)
- net TWI1_SDA: now also J?.18 (Pin_18)
Changed lines of the file:
@@
 	4900 6600 3950 6600
 Wire Wire Line
-	4900 6800 3950 6800
-Wire Wire Line
 	4900 6900 3950 6900
 Wire Wire Line
@@
 F 0 "J1" H 22300 14450 50  0000 L CNN
 F 1 "Conn_01x30" H 22300 14350 50  0000 L CNN
-F 2 "footprint-lib.pretty:Pin_Header_Straight_1x30_Pitch2.54mm" H 22200 14450 50  0001 C CNN
+F 2 "footprint-lib.pretty:Pin_Header_Straight_1x30_Pitch1.27mm" H 22200 14450 50  0001 C CNN
 F 3 "~" H 22200 14450 50  0001 C CNN
 	1    22200 14450
@@
 F 0 "J2" H 25350 14450 50  0000 L CNN
 F 1 "Conn_01x30" H 25350 14350 50  0000 L CNN
-F 2 "footprint-lib.pretty:Pin_Header_Straight_1x30_Pitch2.54mm" H 25250 14450 50  0001 C CNN
+F 2 "footprint-lib.pretty:Pin_Header_Straight_1x30_Pitch1.27mm" H 25250 14450 50  0001 C CNN
 F 3 "~" H 25250 14450 50  0001 C CNN
 	1    25250 14450
@@
 	43700 4400 43700 4300
 Connection ~ 43050 4400
+$Comp
+L Connector_Generic:Conn_01x24 J?
+U 1 1 5DA87EF6
+P 1750 5300
+F 0 "J?" H 1650 3850 50  0000 C CNN
+F 1 "Conn_01x24" H 1650 3950 50  0000 C CNN
+F 2 "" H 1750 5300 50  0001 C CNN
+F 3 "~" H 1750 5300 50  0001 C CNN
+	1    1750 5300
+	-1   0    0    1
+$EndComp
+$Comp
+L customized_power:+5V #PWR?
+U 1 1 5DA8912A
+P 2050 6500
+F 0 "#PWR?" H 2050 6350 50  0001 C CNN
+F 1 "+5V" H 2050 6700 50  0000 C CNN
+F 2 "" H 2050 6500 50  0001 C CNN
+F 3 "" H 2050 6500 50  0001 C CNN
+	1    2050 6500
+	-1   0    0    1
+$EndComp
+Wire Wire Line
+	1950 6400 2050 6400
+Wire Wire Line
+	2050 6400 2050 6500
+$Comp
+L customized_power:+3V3 #PWR?
+U 1 1 5DB30217
+P 2250 6500
+F 0 "#PWR?" H 2250 6350 50  0001 C CNN
+F 1 "+3V3" H 2250 6700 50  0000 C CNN
+F 2 "" H 2250 6500 50  0001 C CNN
+F 3 "" H 2250 6500 50  0001 C CNN
+	1    2250 6500
+	-1   0    0    1
+$EndComp
+Wire Wire Line
+	2250 6500 2250 6300
+Wire Wire Line
+	2250 6300 1950 6300
+$Comp
+L power:GND #PWR?
+U 1 1 5DBD907C
+P 2400 6500
+F 0 "#PWR?" H 2400 6250 50  0001 C CNN
+F 1 "GND" H 2450 6300 50  0000 C CNN
+F 2 "" H 2400 6500 50  0001 C CNN
+F 3 "" H 2400 6500 50  0001 C CNN
+	1    2400 6500
+	1    0    0    -1
+$EndComp
+Wire Wire Line
+	2400 6500 2400 6200
+Wire Wire Line
+	2400 6200 1950 6200
+Text Label 4450 5100 0    50   ~ 0
+CSI_D14
+Text Label 4450 5200 0    50   ~ 0
+CSI_D13
+Text Label 4450 5300 0    50   ~ 0
+CSI_D12
+Text Label 4450 5400 0    50   ~ 0
+CSI_D11
+Text Label 4450 5500 0    50   ~ 0
+CSI_D10
+Text Label 4450 5600 0    50   ~ 0
+CSI_D9
+Text Label 4450 6000 0    50   ~ 0
+CSI_D8
+Text Label 4450 6100 0    50   ~ 0
+CSI_D7
+Text Label 4450 6200 0    50   ~ 0
+CSI_D6
+Text Label 4450 6500 0    50   ~ 0
+CSI_D5
+Text Label 4450 6600 0    50   ~ 0
+CSI_D4
+Wire Wire Line
+	4900 6800 3950 6800
+Text Label 4450 6800 0    50   ~ 0
+CSI_D3
+Text Label 4450 6900 0    50   ~ 0
+CSI_D2
+Text Label 4450 7000 0    50   ~ 0
+CSI_D1
+Text Label 6000 8450 1    50   ~ 0
+CSI_D0
+Text Label 6100 8450 1    50   ~ 0
+CSI_VSYNC
+Text Label 6200 8450 1    50   ~ 0
+CSI_HSYNC
+Text Label 6300 8450 1    50   ~ 0
+CSI_MCLK
+Text Label 6400 8450 1    50   ~ 0
+CSI_PCLK
+Text Label 2650 4300 2    50   ~ 0
+CSI_D12
+Text Label 2650 4400 2    50   ~ 0
+CSI_PCLK
+Text Label 2650 4500 2    50   ~ 0
+CSI_MCLK
+Text Label 2650 4800 2    50   ~ 0
+CSI_HSYNC
+Text Label 2650 4900 2    50   ~ 0
+CSI_VSYNC
+Text Label 2650 5000 2    50   ~ 0
+CSI_D1
+Text Label 2650 5100 2    50   ~ 0
+CSI_D0
+Text Label 2650 5200 2    50   ~ 0
+CSI_D3
+Text Label 2650 5300 2    50   ~ 0
+CSI_D2
+Text Label 2650 5400 2    50   ~ 0
+CSI_D5
+Text Label 2650 5500 2    50   ~ 0
+CSI_D4
+Text Label 2650 5600 2    50   ~ 0
+CSI_D7
+Text Label 2650 5700 2    50   ~ 0
+CSI_D6
+Text Label 2650 5800 2    50   ~ 0
+CSI_D9
+Text Label 2650 5900 2    50   ~ 0
+CSI_D8
+Text Label 2650 6000 2    50   ~ 0
+CSI_D11
+Text Label 2650 6100 2    50   ~ 0
+CSI_D10
+Text Label 7500 8450 1    50   ~ 0
+I2C1_SCL
+Text Label 7600 8450 1    50   ~ 0
+I2C1_SDA
+Text Label 2650 4600 2    50   ~ 0
+I2C1_SCL
+Text Label 2650 4700 2    50   ~ 0
+I2C1_SDA
+Wire Wire Line
+	2650 4300 1950 4300
+Wire Wire Line
+	2650 4400 1950 4400
+Wire Wire Line
+	2650 4500 1950 4500
+Wire Wire Line
+	2650 4600 1950 4600
+Wire Wire Line
+	2650 4700 1950 4700
+Wire Wire Line
+	2650 4800 1950 4800
+Wire Wire Line
+	2650 4900 1950 4900
+Wire Wire Line
+	2650 5000 1950 5000
+Wire Wire Line
+	2650 5100 1950 5100
+Wire Wire Line
+	2650 5200 1950 5200
+Wire Wire Line
+	2650 5300 1950 5300
+Wire Wire Line
+	2650 5400 1950 5400
+Wire Wire Line
+	2650 5500 1950 5500
+Wire Wire Line
+	2650 5600 1950 5600
+Wire Wire Line
+	2650 5700 1950 5700
+Wire Wire Line
+	2650 5800 1950 5800
+Wire Wire Line
+	2650 5900 1950 5900
+Wire Wire Line
+	2650 6000 1950 6000
+Wire Wire Line
+	2650 6100 1950 6100
 $EndSCHEMATC

Commit message: update,
Parts:
- C1, C11, C12, C13, C14, C15, C16, C17, C18, C19, C2, C20, C21, C22, C23, C24, C25, C26, C27, C28, C29, C3, C30, C31, C32, C33, C34, C35, C36, C37, C38, C39, C4, C40, C41, C42, C43, C44, C45, C46, C47, C48, C49, C5, C50, C51, C52, C53, C54, C55, C56, C57, C58, C6, C7, C8: footprint Capacitor_SMD:C_0805_2012Metric_Pad1.15x1.40mm_HandSolder -> Capacitor_SMD:C_0603_1608Metric_Pad1.05x0.95mm_HandSolder
- C59, C60, C61, C62, C63, C64, C65, C66: renamed from C?; footprint (none) -> Capacitor_SMD:C_0603_1608Metric_Pad1.05x0.95mm_HandSolder
- J3: renamed from J?; footprint (none) -> Connector_FFC-FPC:TE_2-84953-4_1x24-1MP_P1.0mm_Horizontal
- L1, L2, L3, L4: footprint Inductor_SMD:L_0805_2012Metric_Pad1.15x1.40mm_HandSolder -> w_smd_inductors:inductor_smd_3x1.4mm
- L5: renamed from L?; footprint (none) -> w_smd_inductors:inductor_smd_3x1.4mm
- MK1: renamed from MK?; footprint (none) -> footprint-lib.pretty:Pin_Header_Straight_1x02_Pitch2.54mm
- R1, R10, R11, R12, R13, R14, R15, R16, R17, R18, R19, R2, R20, R21, R22, R23, R24, R3, R4, R5, R6, R7, R8, R9: footprint Resistor_SMD:R_0805_2012Metric_Pad1.15x1.40mm_HandSolder -> Resistor_SMD:R_0603_1608Metric_Pad1.05x0.95mm_HandSolder
- R29, R30, R31, R32, R33, R34, R35, R36, R37, R38: renamed from R?; footprint (none) -> Resistor_SMD:R_0603_1608Metric_Pad1.05x0.95mm_HandSolder
- SW1, SW2, SW3, SW4: renamed from SW?; footprint (none) -> Button_Switch_SMD:SW_SPST_PTS645
- U4: footprint w_smd_lqfp:lqfp128 -> footprint-lib.pretty:v3s-elqfp128
- gave numbers to parts that had none: 1

Commit message: update,
Changed lines of the file:
@@
 AR Path="/5BCCA602/5BFB14AD" Ref="R?"  Part="1"
 AR Path="/5BCC9E7B/5BFB14AD" Ref="R5"  Part="1"
-F 0 "R5" H 22300 4700 50  0000 L CNN
-F 1 "R473" H 22300 4650 50  0000 L CNN
+F 0 "R5" H 22100 4700 50  0000 R CNN
+F 1 "R473" H 22100 4650 50  0000 R CNN
 F 2 "Resistor_SMD:R_0603_1608Metric_Pad1.05x0.95mm_HandSolder" H 22200 4650 50  0001 C CNN
 F 3 "~" H 22200 4650 50  0001 C CNN
@@
 U 1 1 5C4CCCAA
 P 33950 2150
-F 0 "R33" V 33700 2150 50  0000 C CNN
-F 1 "R510" V 33800 2150 50  0000 C CNN
+F 0 "R33" V 34100 2150 50  0000 C CNN
+F 1 "R510" V 34200 2150 50  0000 C CNN
 F 2 "Resistor_SMD:R_0603_1608Metric_Pad1.05x0.95mm_HandSolder" H 33950 2150 50  0001 C CNN
 F 3 "~" H 33950 2150 50  0001 C CNN
