File: allwinner-v3s-tryout.kicad_pcb (KiCad board)
At the start: 2 copper layers, 90 x 60 mm, 0 parts

Commit message: update,
Parts:
- added C1: C106, Capacitor_SMD:C_0603_1608Metric_Pad1.05x0.95mm_HandSolder, F.Cu at (42.0, 49.4)
- added C10: C104-50v, Capacitor_SMD:C_1206_3216Metric_Pad1.42x1.75mm_HandSolder, F.Cu at (36.5, 29.4)
- added C11: C106, Capacitor_SMD:C_0603_1608Metric_Pad1.05x0.95mm_HandSolder, F.Cu at (63.6, 36.0)
- added C12: C18pf, Capacitor_SMD:C_0603_1608Metric_Pad1.05x0.95mm_HandSolder, F.Cu at (59.8, 36.9)
- added C13: C18pf, Capacitor_SMD:C_0603_1608Metric_Pad1.05x0.95mm_HandSolder, F.Cu at (59.8, 40.8)
- added C14: C106, Capacitor_SMD:C_0603_1608Metric_Pad1.05x0.95mm_HandSolder, F.Cu at (56.1, 44.7)
- added C15: C105, Capacitor_SMD:C_0603_1608Metric_Pad1.05x0.95mm_HandSolder, F.Cu at (72.7, 29.0)
- added C16: C105, Capacitor_SMD:C_0603_1608Metric_Pad1.05x0.95mm_HandSolder, F.Cu at (63.6, 38.0)
- added C17: C104, Capacitor_SMD:C_0603_1608Metric_Pad1.05x0.95mm_HandSolder, F.Cu at (76.4, 24.7)
- added C18: C104, Capacitor_SMD:C_0603_1608Metric_Pad1.05x0.95mm_HandSolder, F.Cu at (76.4, 26.7)
- added C19: C106, Capacitor_SMD:C_0603_1608Metric_Pad1.05x0.95mm_HandSolder, F.Cu at (76.4, 20.8)
- added C2: C104, Capacitor_SMD:C_0603_1608Metric_Pad1.05x0.95mm_HandSolder, F.Cu at (56.1, 40.8)
- added C20: C105, Capacitor_SMD:C_0603_1608Metric_Pad1.05x0.95mm_HandSolder, F.Cu at (56.1, 46.7)
- added C21: C105, Capacitor_SMD:C_0603_1608Metric_Pad1.05x0.95mm_HandSolder, F.Cu at (59.8, 42.8)
- added C22: C104, Capacitor_SMD:C_0603_1608Metric_Pad1.05x0.95mm_HandSolder, F.Cu at (53.3, 48.6)
- added C23: C104, Capacitor_SMD:C_0603_1608Metric_Pad1.05x0.95mm_HandSolder, F.Cu at (71.1, 31.0)
- added C24: C104, Capacitor_SMD:C_0603_1608Metric_Pad1.05x0.95mm_HandSolder, F.Cu at (56.1, 33.0)
- added C25: C106, Capacitor_SMD:C_0603_1608Metric_Pad1.05x0.95mm_HandSolder, F.Cu at (76.4, 22.8)
- added C26: C104, Capacitor_SMD:C_0603_1608Metric_Pad1.05x0.95mm_HandSolder, F.Cu at (67.3, 36.0)
- added C27: C106, Capacitor_SMD:C_0603_1608Metric_Pad1.05x0.95mm_HandSolder, F.Cu at (67.3, 32.1)
- added C28: C106, Capacitor_SMD:C_0603_1608Metric_Pad1.05x0.95mm_HandSolder, F.Cu at (67.3, 34.1)
- added C29: C104, Capacitor_SMD:C_0603_1608Metric_Pad1.05x0.95mm_HandSolder, F.Cu at (63.6, 34.1)
- added C3: C104, Capacitor_SMD:C_0603_1608Metric_Pad1.05x0.95mm_HandSolder, F.Cu at (76.4, 15.0)
- added C30: C106, Capacitor_SMD:C_0603_1608Metric_Pad1.05x0.95mm_HandSolder, F.Cu at (72.7, 25.1)
- added C31: C105, Capacitor_SMD:C_0603_1608Metric_Pad1.05x0.95mm_HandSolder, F.Cu at (59.8, 38.9)
- added C32: C104, Capacitor_SMD:C_0603_1608Metric_Pad1.05x0.95mm_HandSolder, F.Cu at (56.1, 42.8)
- added C33: C104, Capacitor_SMD:C_0603_1608Metric_Pad1.05x0.95mm_HandSolder, F.Cu at (52.3, 46.7)
- added C34: C106, Capacitor_SMD:C_0603_1608Metric_Pad1.05x0.95mm_HandSolder, F.Cu at (68.9, 29.0)
- added C35: C105, Capacitor_SMD:C_0603_1608Metric_Pad1.05x0.95mm_HandSolder, F.Cu at (56.1, 38.9)
- added C36: C104, Capacitor_SMD:C_0603_1608Metric_Pad1.05x0.95mm_HandSolder, F.Cu at (56.1, 35.0)
- added C37: C104, Capacitor_SMD:C_0603_1608Metric_Pad1.05x0.95mm_HandSolder, F.Cu at (59.8, 35.0)
- added C38: C104, Capacitor_SMD:C_0603_1608Metric_Pad1.05x0.95mm_HandSolder, F.Cu at (63.6, 32.1)
- added C39: C104, Capacitor_SMD:C_0603_1608Metric_Pad1.05x0.95mm_HandSolder, F.Cu at (72.7, 23.2)
- added C4: C102, Capacitor_SMD:C_0603_1608Metric_Pad1.05x0.95mm_HandSolder, F.Cu at (59.8, 33.0)
- added C40: C104, Capacitor_SMD:C_0603_1608Metric_Pad1.05x0.95mm_HandSolder, F.Cu at (68.9, 27.1)
- added C41: C104, Capacitor_SMD:C_0603_1608Metric_Pad1.05x0.95mm_HandSolder, F.Cu at (45.8, 49.4)
- added C42: C104, Capacitor_SMD:C_0603_1608Metric_Pad1.05x0.95mm_HandSolder, F.Cu at (68.9, 25.1)
- added C43: C106, Capacitor_SMD:C_0603_1608Metric_Pad1.05x0.95mm_HandSolder, F.Cu at (72.7, 21.2)
- added C44: C105, Capacitor_SMD:C_0603_1608Metric_Pad1.05x0.95mm_HandSolder, F.Cu at (76.4, 18.9)
- added C45: C105, Capacitor_SMD:C_0603_1608Metric_Pad1.05x0.95mm_HandSolder, F.Cu at (52.3, 42.8)
- added C46: C104, Capacitor_SMD:C_0603_1608Metric_Pad1.05x0.95mm_HandSolder, F.Cu at (65.2, 26.3)
- added C47: C104, Capacitor_SMD:C_0603_1608Metric_Pad1.05x0.95mm_HandSolder, F.Cu at (73.2, 13.0)
- added C48: C106, Capacitor_SMD:C_0603_1608Metric_Pad1.05x0.95mm_HandSolder, F.Cu at (52.3, 40.8)
- added C49: C18pf, Capacitor_SMD:C_0603_1608Metric_Pad1.05x0.95mm_HandSolder, F.Cu at (56.1, 36.9)
- added C5: C105, Capacitor_SMD:C_0603_1608Metric_Pad1.05x0.95mm_HandSolder, F.Cu at (68.9, 23.2)
- added C50: C106, Capacitor_SMD:C_0603_1608Metric_Pad1.05x0.95mm_HandSolder, F.Cu at (77.0, 13.0)
- added C51: C106, Capacitor_SMD:C_0603_1608Metric_Pad1.05x0.95mm_HandSolder, F.Cu at (52.3, 44.7)
- added C52: C106, Capacitor_SMD:C_0603_1608Metric_Pad1.05x0.95mm_HandSolder, F.Cu at (72.7, 27.1)
- added C53: C18pf, Capacitor_SMD:C_0603_1608Metric_Pad1.05x0.95mm_HandSolder, F.Cu at (52.3, 38.9)
- added C54: C106, Capacitor_SMD:C_0603_1608Metric_Pad1.05x0.95mm_HandSolder, F.Cu at (65.2, 30.2)
- added C55: C106, Capacitor_SMD:C_0603_1608Metric_Pad1.05x0.95mm_HandSolder, F.Cu at (49.5, 49.4)
- added C56: C18pf, Capacitor_SMD:C_0603_1608Metric_Pad1.05x0.95mm_HandSolder, F.Cu at (68.9, 21.2)
- added C57: C104, Capacitor_SMD:C_0603_1608Metric_Pad1.05x0.95mm_HandSolder, F.Cu at (30.2, 45.2)
- added C58: C106, Capacitor_SMD:C_0603_1608Metric_Pad1.05x0.95mm_HandSolder, F.Cu at (65.2, 28.2)
- added C59: C105, Capacitor_SMD:C_0603_1608Metric_Pad1.05x0.95mm_HandSolder, F.Cu at (89.7, 37.7)
- added C6: C104, Capacitor_SMD:C_0603_1608Metric_Pad1.05x0.95mm_HandSolder, F.Cu at (72.7, 19.3)
- added C60: C104, Capacitor_SMD:C_0603_1608Metric_Pad1.05x0.95mm_HandSolder, F.Cu at (93.1, 37.7)
- added C61: C33pf, Capacitor_SMD:C_0603_1608Metric_Pad1.05x0.95mm_HandSolder, F.Cu at (96.4, 37.7)
- added C62: C104, Capacitor_SMD:C_0603_1608Metric_Pad1.05x0.95mm_HandSolder, F.Cu at (99.8, 37.7)
- added C63: C104, Capacitor_SMD:C_0603_1608Metric_Pad1.05x0.95mm_HandSolder, F.Cu at (103.1, 37.7)
- added C64: C101, Capacitor_SMD:C_0603_1608Metric_Pad1.05x0.95mm_HandSolder, F.Cu at (89.7, 39.2)
- added C65: C33pf, Capacitor_SMD:C_0603_1608Metric_Pad1.05x0.95mm_HandSolder, F.Cu at (96.4, 39.2)
- added C66: C104, Capacitor_SMD:C_0603_1608Metric_Pad1.05x0.95mm_HandSolder, F.Cu at (93.1, 39.2)
- added C7: C18pf, Capacitor_SMD:C_0603_1608Metric_Pad1.05x0.95mm_HandSolder, F.Cu at (76.4, 16.9)
- added C8: C18pf, Capacitor_SMD:C_0603_1608Metric_Pad1.05x0.95mm_HandSolder, F.Cu at (68.9, 19.3)
- added C9: C106-50v, Capacitor_SMD:C_1206_3216Metric_Pad1.42x1.75mm_HandSolder, F.Cu at (22.1, 45.3)
- added D1: SD_1N5819_S4, Diode_SMD:D_SOD-123F, F.Cu at (26.7, 47.7)
- added J1: Conn_01x30, footprint-lib.pretty:Pin_Header_Straight_1x30_Pitch1.27mm, F.Cu at (7.32, 47.2)
- added J2: Conn_01x30, footprint-lib.pretty:Pin_Header_Straight_1x30_Pitch1.27mm, F.Cu at (93.4, 7.57)
- added J3: Conn_01x24, Connector_FFC-FPC:TE_2-84953-4_1x24-1MP_P1.0mm_Horizontal, F.Cu at (97.4, 29.9)
- added L1: L_2.2uH, w_smd_inductors:inductor_smd_3x1.4mm, F.Cu at (72.7, 17.3)
- added L2: L_2.2uH, w_smd_inductors:inductor_smd_3x1.4mm, F.Cu at (65.2, 24.3)
- added L3: L_2.2uH, w_smd_inductors:inductor_smd_3x1.4mm, F.Cu at (72.7, 15.4)
- added L4: L_2.2uH, w_smd_inductors:inductor_smd_3x1.4mm, F.Cu at (52.3, 36.9)
- added L5: L_10uH, w_smd_inductors:inductor_smd_3x1.4mm, F.Cu at (86.3, 38.7)
- added MK1: Microphone, footprint-lib.pretty:Pin_Header_Straight_1x02_Pitch2.54mm, F.Cu at (82.7, 38.8)
- added R1: R473, Resistor_SMD:R_0603_1608Metric_Pad1.05x0.95mm_HandSolder, F.Cu at (68.9, 15.4)
- added R10: R473, Resistor_SMD:R_0603_1608Metric_Pad1.05x0.95mm_HandSolder, F.Cu at (61.4, 30.2)
- added R11: R106, Resistor_SMD:R_0603_1608Metric_Pad1.05x0.95mm_HandSolder, F.Cu at (31.3, 37.7)
- added R12: R103, Resistor_SMD:R_0603_1608Metric_Pad1.05x0.95mm_HandSolder, F.Cu at (65.2, 18.5)
- added R13: R5R1, Resistor_SMD:R_0603_1608Metric_Pad1.05x0.95mm_HandSolder, F.Cu at (61.4, 22.4)
- added R14: R103, Resistor_SMD:R_0603_1608Metric_Pad1.05x0.95mm_HandSolder, F.Cu at (52.3, 33.0)
- added R15: R0, Resistor_SMD:R_0603_1608Metric_Pad1.05x0.95mm_HandSolder, F.Cu at (61.4, 20.4)
- added R16: R204, Resistor_SMD:R_0603_1608Metric_Pad1.05x0.95mm_HandSolder, F.Cu at (61.4, 18.5)
- added R17: R202, Resistor_SMD:R_0603_1608Metric_Pad1.05x0.95mm_HandSolder, F.Cu at (30.8, 49.4)
- added R18: R202, Resistor_SMD:R_0603_1608Metric_Pad1.05x0.95mm_HandSolder, F.Cu at (65.2, 16.5)
- added R19: R684, Resistor_SMD:R_0603_1608Metric_Pad1.05x0.95mm_HandSolder, F.Cu at (61.4, 16.5)
- added R2: R241, Resistor_SMD:R_0603_1608Metric_Pad1.05x0.95mm_HandSolder, F.Cu at (30.8, 43.3)
- added R20: R154, Resistor_SMD:R_0603_1608Metric_Pad1.05x0.95mm_HandSolder, F.Cu at (52.3, 35.0)
- added R21: R684, Resistor_SMD:R_0603_1608Metric_Pad1.05x0.95mm_HandSolder, F.Cu at (77.0, 11.1)
- added R22: R154, Resistor_SMD:R_0603_1608Metric_Pad1.05x0.95mm_HandSolder, F.Cu at (61.4, 26.3)
- added R23: R684, Resistor_SMD:R_0603_1608Metric_Pad1.05x0.95mm_HandSolder, F.Cu at (65.2, 22.4)
- added R24: R154, Resistor_SMD:R_0603_1608Metric_Pad1.05x0.95mm_HandSolder, F.Cu at (68.9, 17.3)
- added R25: R202, Resistor_SMD:R_0603_1608Metric_Pad1.05x0.95mm_HandSolder, F.Cu at (59.6, 44.5)
- added R26: R202, Resistor_SMD:R_0603_1608Metric_Pad1.05x0.95mm_HandSolder, F.Cu at (70.9, 32.7)
- added R27: R202, Resistor_SMD:R_0603_1608Metric_Pad1.05x0.95mm_HandSolder, F.Cu at (63.4, 39.7)
- added R28: R202, Resistor_SMD:R_0603_1608Metric_Pad1.05x0.95mm_HandSolder, F.Cu at (26.1, 49.6)
- added R29: R510, Resistor_SMD:R_0603_1608Metric_Pad1.05x0.95mm_HandSolder, F.Cu at (95.2, 50.4)
- added R3: R602, Resistor_SMD:R_0603_1608Metric_Pad1.05x0.95mm_HandSolder, F.Cu at (73.2, 11.1)
- added R30: R202, Resistor_SMD:R_0603_1608Metric_Pad1.05x0.95mm_HandSolder, F.Cu at (98.6, 47.4)
- added R31: R510, Resistor_SMD:R_0603_1608Metric_Pad1.05x0.95mm_HandSolder, F.Cu at (95.2, 51.9)
- added R32: R510, Resistor_SMD:R_0603_1608Metric_Pad1.05x0.95mm_HandSolder, F.Cu at (95.2, 48.9)
- added R33: R510, Resistor_SMD:R_0603_1608Metric_Pad1.05x0.95mm_HandSolder, F.Cu at (95.2, 47.4)
- added R34: R202, Resistor_SMD:R_0603_1608Metric_Pad1.05x0.95mm_HandSolder, F.Cu at (98.6, 45.8)
- added R35: R682, Resistor_SMD:R_0603_1608Metric_Pad1.05x0.95mm_HandSolder, F.Cu at (81.6, 59.5)
- added R36: R822, Resistor_SMD:R_0603_1608Metric_Pad1.05x0.95mm_HandSolder, F.Cu at (78.3, 59.5)
- added R37: R103, Resistor_SMD:R_0603_1608Metric_Pad1.05x0.95mm_HandSolder, F.Cu at (95.2, 45.8)
- added R38: R113, Resistor_SMD:R_0603_1608Metric_Pad1.05x0.95mm_HandSolder, F.Cu at (74.9, 59.5)
- added R4: R104, Resistor_SMD:R_0603_1608Metric_Pad1.05x0.95mm_HandSolder, F.Cu at (61.4, 24.3)
- added R5: R473, Resistor_SMD:R_0603_1608Metric_Pad1.05x0.95mm_HandSolder, F.Cu at (65.2, 20.4)
- added R6: R473, Resistor_SMD:R_0603_1608Metric_Pad1.05x0.95mm_HandSolder, F.Cu at (26.4, 45.2)
- added R7: R473, Resistor_SMD:R_0603_1608Metric_Pad1.05x0.95mm_HandSolder, F.Cu at (38.3, 49.4)
- added R8: R473, Resistor_SMD:R_0603_1608Metric_Pad1.05x0.95mm_HandSolder, F.Cu at (61.4, 28.2)
- added R9: R473, Resistor_SMD:R_0603_1608Metric_Pad1.05x0.95mm_HandSolder, F.Cu at (34.5, 49.4)
- added SW1: SW_Push, Button_Switch_SMD:SW_SPST_PTS645, F.Cu at (78.3, 55.4)
- added SW2: SW_Push, Button_Switch_SMD:SW_SPST_PTS645, F.Cu at (78.3, 48.5)
- added SW3: SW_Push, Button_Switch_SMD:SW_SPST_PTS645, F.Cu at (88.5, 48.5)
- added SW4: SW_Push, Button_Switch_SMD:SW_SPST_PTS645, F.Cu at (88.5, 55.4)
- added U1: USB_MICRO, Connector_PinHeader_2.54mm:PinHeader_1x05_P2.54mm_Vertical, F.Cu at (17.8, 38.5)
- added U10: GD5F1GQ4UAYIG, Package_SO:SOIC-8_3.9x4.9mm_P1.27mm, F.Cu at (23.3, 41.5)
- added U11: EA3036, Package_DFN_QFN:QFN-24-1EP_3x3mm_P0.4mm_EP1.75x1.6mm_ThermalVias, F.Cu at (69.2, 12.3)
- added U12: XC6206, Package_TO_SOT_SMD:SOT-23_Handsoldering, F.Cu at (29.8, 40.5)
- added U13: HR911105A, footprint-lib.pretty:HANRUN_HR911105A, F.Cu at (46.5, 8.46)
- added U2: NS2009, Package_SO:MSOP-10_3x3mm_P0.5mm, F.Cu at (37.2, 22.0)
- added U3: FC-40P-LCD, footprint-lib.pretty:HIROSE_FH12S-40S-0.5SH(55), F.Cu at (23.1, 14.1)
- added U4: allwinner-V3S-eLQFP128, footprint-lib.pretty:v3s-elqfp128, F.Cu at (24.7, 26.1)
- added U5: TF_CARD, footprint-lib.pretty:SUNTECH_ST-TF-003A, F.Cu at (24.2, 56.4)
- added U6: MC-146, Crystal:Crystal_SMD_SeikoEpson_MC146-4Pin_6.7x1.5mm_HandSoldering, F.Cu at (24.5, 37.7)
- added U7: MX25L12835F, Package_SO:SOIC-8_3.9x4.9mm_P1.27mm, F.Cu at (63.3, 12.8)
- added U8: PT4101, Package_TO_SOT_SMD:SOT-23-6_Handsoldering, F.Cu at (22.0, 48.3)
- added U9: XT_3225, Crystal:Crystal_SMD_SeikoEpson_TSX3225-4Pin_3.2x2.5mm_HandSoldering, F.Cu at (36.9, 26.1)

Commit message: update,
Parts:
- removed J1, J2: Conn_01x30, footprint-lib.pretty:Pin_Header_Straight_1x30_Pitch1.27mm
- removed J3: Conn_01x24, Connector_FFC-FPC:TE_2-84953-4_1x24-1MP_P1.0mm_Horizontal
- C1, C10, C11, C14, C15, C16, C17, C18, C19, C2, C20, C21, C22, C24, C32, C33, C34, C35, C36, C38, C41, C42, C58, C9, D1, L1, R1, R12, R13, R17, R18, R2, R25, R26, R27, R28, R5, R6, R7, R8, R9, U10, U2, U7, U8: moved to B.Cu
- moved C37 125.8 mm to (185.6, 38.5)
- moved L4 108.6 mm to (153.5, 76.3), turned to 90 degrees
- moved C51 108.0 mm to (159.5, 58.1), turned to 270 degrees
- moved U11 104.2 mm to (159.5, 64.2), turned to 180 degrees
- moved C53 101.7 mm to (149.2, 69.7), turned to 270 degrees
- moved R24 100.2 mm to (146.6, 80.6)
- moved R20 98.7 mm to (145.9, 66.3)
- moved C55 98.5 mm to (143.9, 77.6), turned to 270 degrees
- moved R4 98.1 mm to (140.3, 82.6), turned to 270 degrees
- moved R23 97.7 mm to (145.8, 77.6), turned to 270 degrees
- moved C56 97.5 mm to (148.5, 77.6), turned to 270 degrees
- moved R22 97.4 mm to (147.0, 72.8)
- moved C4 96.7 mm to (140.2, 86.8), turned to 270 degrees
- moved C54 96.7 mm to (157.7, 58.1), turned to 270 degrees
- moved C49 96.4 mm to (148.7, 63.5), turned to 270 degrees
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Routing:
- net GND: track 0.00 -> 365.0 mm, vias 0 -> 1
- net +3V3: track 0.00 -> 94.6 mm, vias 0 -> 6
- net +1V2: track 0.00 -> 85.2 mm, vias 0 -> 10
- net +5V: track 0.00 -> 51.3 mm
- net LCD_D4: track 0.00 -> 36.4 mm, vias 0 -> 2
- net LCD_D3: track 0.00 -> 32.2 mm, vias 0 -> 2
- net LCD_DE: track 0.00 -> 31.9 mm, vias 0 -> 2
- net LCD_HSYNC: track 0.00 -> 31.7 mm, vias 0 -> 2
- net LCD_D2: track 0.00 -> 29.9 mm, vias 0 -> 2
- net VLED+: track 0.00 -> 28.9 mm, vias 0 -> 3
- net LCD_D21: track 0.00 -> 26.3 mm, vias 0 -> 2
- net LCD_D18: track 0.00 -> 25.3 mm
- net LCD_D20: track 0.00 -> 24.6 mm, vias 0 -> 2
- net LCD_D10: track 0.00 -> 24.6 mm, vias 0 -> 2
- net LCD_D19: track 0.00 -> 24.4 mm, vias 0 -> 2
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Other:
- board size 90 x 60 mm -> 100 x 70 mm
- net class Default: clearance 0.2 -> 0.1; trace_width 0.25 -> 0.2
- rule trace_clearance: 0.2 -> 0.1
